Commit message: updated velocity timeout

File: naviclean_description/urdf/naviclean.xacro (robot description, xacro)
@@ -25,5 +25,5 @@
       <mesh filename="package://naviclean_description/meshes/base_link.stl" scale="0.001 0.001 0.001"/>
     </geometry> -->
-    <origin xyz="0.0 0 0.005" rpy="0 0 0"/>
+    <origin xyz="0.0 0 0.006" rpy="0 0 0"/>
     <geometry>
       <box size="0.35 0.25 0.0085" />

Commit message: Updated urdf for lidar frame fix

File: naviclean_description/urdf/naviclean.xacro (robot description, xacro)
@@ -84,5 +84,5 @@
   </inertial>
   <visual>
-    <origin xyz="0.0 0.0 -0.335" rpy="0 0 3.1416"/>
+    <origin xyz="0.0 0.0 -0.335" rpy="0 0 0"/>
     <geometry>
       <mesh filename="package://naviclean_description/meshes/ydlidar_1.stl" scale="0.001 0.001 0.001"/>
@@ -91,5 +91,5 @@
   </visual>
   <collision>
-    <origin xyz="0.0 0.0 -0.335" rpy="0 0 3.1416"/>
+    <origin xyz="0.0 0.0 -0.335" rpy="0 0 0"/>
     <geometry>
       <mesh filename="package://naviclean_description/meshes/ydlidar_1.stl" scale="0.001 0.001 0.001"/>
@@ -110,5 +110,5 @@
 </joint>
 <joint name="base2lidar" type="fixed">
-  <origin xyz="-0.0 -0.0 0.335" rpy="0 0 3.1416"/>
+  <origin xyz="-0.0 -0.0 0.335" rpy="0 0 0"/>
   <parent link="base_link"/>
   <child link="ydlidar_1"/>
